Commit message: fix file names

File: jcb_description/urdf/jcb_description.urdf (robot description, URDF)
Before this commit: robot jcb3, 5 links, 4 joints
Links:
- link Link_1: geometry collision mesh filename=package://jcb_description/meshes/Link_1.STL; visual mesh filename=package://jcb_description/meshes/Link_1.STL
- link Link_2: geometry collision mesh filename=package://jcb_description/meshes/Link_2.STL; visual mesh filename=package://jcb_description/meshes/Link_2.STL
- link Link_3: geometry collision mesh filename=package://jcb_description/meshes/Link_3.STL; visual mesh filename=package://jcb_description/meshes/Link_3.STL
- link base_link: geometry collision mesh filename=package://jcb_description/meshes/base_link.STL; visual mesh filename=package://jcb_description/meshes/base_link.STL
